Commit message: remove franka gripper to make meshcat work for now

File: assets/franka_panda_urdf/panda.urdf (robot description, URDF)
Before this commit: robot panda, 12 links, 11 joints
Links:
- removed link panda_hand
- removed link panda_leftfinger
- removed link panda_rightfinger
- link panda_link0: geometry collision mesh filename=package://meshes/collision/link0.obj; visual mesh filename=package://meshes/collision/link0.obj
- link panda_link1: geometry collision mesh filename=package://meshes/collision/link1.obj; visual mesh filename=package://meshes/collision/link1.obj
- link panda_link2: geometry collision mesh filename=package://meshes/collision/link2.obj; visual mesh filename=package://meshes/collision/link2.obj
- link panda_link3: geometry collision mesh filename=package://meshes/collision/link3.obj; visual mesh filename=package://meshes/collision/link3.obj
- link panda_link4: geometry collision mesh filename=package://meshes/collision/link4.obj; visual mesh filename=package://meshes/collision/link4.obj
- link panda_link5: geometry collision mesh filename=package://meshes/collision/link5.obj; visual mesh filename=package://meshes/collision/link5.obj
- link panda_link6: geometry collision mesh filename=package://meshes/collision/link6.obj; visual mesh filename=package://meshes/collision/link6.obj
- link panda_link7: geometry collision mesh filename=package://meshes/collision/link7.obj; visual mesh filename=package://meshes/collision/link7.obj
Joints:
- removed joint panda_finger_joint1
- removed joint panda_finger_joint2
- removed joint panda_hand_joint
